File: RPI4_is2Power/RPI4_is2Power.kicad_sch (KiCad schematic)
At the start: 25 parts, among them J1 GPIO, J10 5v pin, J11 5v pin, J12 5v pin, J2 Conn_01x03_Socket, J3 U.FL-R-SMT-1_80_, J4 U.FL-R-SMT-1_80_, J5 U.FL-R-SMT-1_80_, J6 U.FL-R-SMT-1_80_, J7 U.FL-R-SMT-1_80_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

Commit message: updated final four boards for streamer
Parts:
- removed C4, C5, C6, C7: 470u, Capacitor_THT:CP_Radial_D10.0mm_P5.00mm, symbol Device:C_Polarized
- removed J10, J11, J12: 5v pin, Connector_Pin:Pin_D0.7mm_L6.5mm_W1.8mm_FlatFork, symbol Connector:Conn_01x01_Pin
- removed J2: Conn_01x03_Socket, samsys:PCB Wired Socket, symbol Connector:Conn_01x03_Socket
- added C1, C4, C5, C6: 330u, CAPPRD350W60D800H1300, symbol NewSamsys:RNU1C331MDN1KX
- added H1, H2, H3, H4: MountingHole, MountingHole:MountingHole_2.5mm, symbol Mechanical:MountingHole
- added J2: 1725669, 1725669, symbol NewSamsys:1725669
- J8, J9: value 5v pin -> Conn_01x01_Pin; footprint Connector_Pin:Pin_D0.7mm_L6.5mm_W1.8mm_FlatFork -> Connector_Pin:Pin_D1.2mm_L11.3mm_W3.0mm_Flat
Connections:
- net +5V: now also C1.1 (+), C4.1 (+), C5.1 (+), C6.1 (+), J2.1, J2.2
- net GND: now also C1.2 (-), C4.2 (-), C5.2 (-), C6.2 (-), J2.3
- no-connect marks 25 -> 26
Other:
- note added: "Mounting Holes"
