File: se_to_diff board/se_to_diff board.kicad_pcb (KiCad board)
At the start: 4 copper layers, 65 x 56.5 mm, 40 parts, among them IC1 1646S08-U, IC2 1646S08-U, J1 1725669, J2 1725669, J3 1725669, J4 1725669

Commit message: updated final four boards for streamer
Parts:
- moved D2 1.53 mm to (123.6, 54.4)
- moved R2 1.53 mm to (123.7, 58.8)
Routing:
- net VEE: track 72.2 -> 74.3 mm
Other:
- board text added: "-5v G +5v"
- board text added: "Input"
- board text added: "L- G L+"
- board text added: "Output"
- board text added: "R G L"
- board text added: "R- G R+"
- board text added: "Riverbank systems Single to Balanced version 0.1"
Changed lines of the file:
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@@
 	(footprint "samsys:LEDC2012X40N"
 		(layer "F.Cu")
-		(at 125.15 54.375 -90)
+		(at 123.625 54.4375 -90)
 		(descr "LS R976")
 		(tags "LED")
@@
 	(footprint "samsys:ERJH3"
 		(layer "F.Cu")
-		(at 125.175 58.75 -90)
+		(at 123.65 58.8125 -90)
 		(descr "ERJH3")
 		(tags "Resistor")
@@
 	)
 	(gr_rect
+		(start 109.875 97.325)
+		(end 124.625 102.2)
+		(stroke
+			(width 0.1)
+			(type default)
+		)
+		(fill none)
+		(layer "F.SilkS")
+	)
+	(gr_rect
 		(start 100 50)
 		(end 165 106.5)
@@
 		(layer "Edge.Cuts")
 	)
+	(gr_text "R- G  R+"
+		(at 162.675 87.3 270)
+		(layer "F.SilkS" knockout)
+		(effects
+			(font
+				(size 1 1)
+				(thickness 0.1)
+				(bold yes)
+			)
+			(justify left bottom)
+		)
+	)
+	(gr_text "-5v G +5v"
+		(at 108.9 52.25 0)
+		(layer "F.SilkS" knockout)
+		(effects
+			(font
+				(size 1 1)
+				(thickness 0.1)
+				(bold yes)
+			)
+			(justify left bottom)
+		)
+	)
+	(gr_text "Output"
+		(at 155.925 71.125 0)
+		(layer "F.SilkS")
+		(effects
+			(font
+				(size 1 1)
+				(thickness 0.1)
+			)
+			(justify left bottom)
+		)
+	)
+	(gr_text "L- G  L+"
+		(at 162.675 73.95 -90)
+		(layer "F.SilkS" knockout)
+		(effects
+			(font
+				(size 1 1)
+				(thickness 0.1)
+				(bold yes)
+			)
+			(justify left bottom)
+		)
+	)
+	(gr_text "Input"
+		(at 105.075 75.725 0)
+		(layer "F.SilkS")
+		(effects
+			(font
+				(size 1 1)
+				(thickness 0.1)
+			)
+			(justify left bottom)
+		)
+	)
+	(gr_text "Riverbank systems \nSingle to Balanced\nversion 0.1"
+		(at 110 102 0)
+		(layer "F.SilkS" knockout)
+		(effects
+			(font
+				(size 1 1)
+				(thickness 0.1)
+			)
+			(justify left bottom)
+		)
+	)
+	(gr_text "R  G  L"
+		(at 102.575 84.675 90)
+		(layer "F.SilkS" knockout)
+		(effects
+			(font
+				(size 1 1)
+				(thickness 0.1)
+				(bold yes)
+			)
+			(justify left bottom)
+		)
+	)
 	(segment
 		(start 141.725 81.2)
@@
 	)
 	(segment
-		(start 125.175 59.475)
-		(end 125.175 61.8)
+		(start 123.65 59.5375)
+		(end 123.65 61.8625)
 		(width 0.5)
 		(layer "F.Cu")
@@
 	)
 	(via
-		(at 125.175 61.8)
+		(at 123.65 61.8625)
 		(size 0.6)
 		(drill 0.3)
@@
 	)
 	(segment
-		(start 135.415 94.555)
-		(end 135.195 96.925)
-		(width 0.5)
-		(layer "F.Cu")
-		(net 7)
-	)
-	(segment
 		(start 137.55 83.625)
 		(end 137.5 83.675)
@@
 	)
 	(segment
+		(start 135.425 94.565)
+		(end 135.425 96.695)
+		(width 0.5)
+		(layer "F.Cu")
+		(net 7)
+	)
+	(segment
 		(start 126.025 51.3)
 		(end 144.925 51.45)
@@
 	)
 	(segment
+		(start 135.415 94.555)
+		(end 135.425 94.565)
+		(width 0.5)
+		(layer "F.Cu")
+		(net 7)
+	)
+	(segment
 		(start 137.5 83.675)
 		(end 135.435 83.675)
@@
 	)
 	(segment
-		(start 120.275 51.925)
-		(end 126.025 51.3)
+		(start 135.425 96.695)
+		(end 135.195 96.925)
 		(width 0.5)
 		(layer "F.Cu")
@@
 	)
 	(segment
-		(start 135.415 81.355)
-		(end 135.415 83.655)
+		(start 120.275 51.925)
+		(end 126.025 51.3)
 		(width 0.5)
 		(layer "F.Cu")
@@
 	)
 	(segment
-		(start 137.395735 96.925)
-		(end 137.525 96.795735)
+		(start 135.415 81.355)
+		(end 135.415 83.655)
 		(width 0.5)
 		(layer "F.Cu")
@@
 	)
 	(segment
-		(start 135.195 96.925)
-		(end 137.395735 96.925)
+		(start 137.395735 96.925)
+		(end 135.195 96.925)
 		(width 0.5)
 		(layer "F.Cu")
@@
 	)
 	(via
-		(at 137.525 96.795735)
+		(at 137.395735 96.925)
 		(size 0.6)
 		(drill 0.3)
@@
 	(segment
 		(start 137.525 83.65)
-		(end 137.525 96.795735)
+		(end 137.55 83.625)
 		(width 0.5)
 		(layer "B.Cu")
@@
 	)
 	(segment
+		(start 137.525 96.795735)
+		(end 137.525 83.65)
+		(width 0.5)
+		(layer "B.Cu")
+		(net 7)
+	)
+	(segment
 		(start 137.55 71.95)
 		(end 144.725 68.4)
@@
 	)
 	(segment
-		(start 137.55 83.625)
-		(end 137.525 83.65)
+		(start 137.395735 96.925)
+		(end 137.525 96.795735)
 		(width 0.5)
 		(layer "B.Cu")
@@
 	)
 	(segment
-		(start 125.15 53.425)
-		(end 129.275 55.025)
+		(start 120.075 59.275)
+		(end 120.075 55.575)
+		(width 0.5)
+		(layer "F.Cu")
+		(net 8)
+	)
+	(segment
+		(start 122.075 53.575)
+		(end 123.625 53.4875)
+		(width 0.5)
+		(layer "F.Cu")
+		(net 8)
+	)
+	(segment
+		(start 129.925 94.8)
+		(end 130.025 94.9)
 		(width 0.5)
 		(layer "F.Cu")
@@
 	)
 	(segment
-		(start 119.8 59)
-		(end 122.775 54.45)
+		(start 113.645 59.275)
+		(end 120.075 59.275)
 		(width 0.5)
 		(layer "F.Cu")
@@
 	)
 	(segment
-		(start 131.875 94.9)
+		(start 134.14 94.55)
 		(end 134.145 94.555)
 		(width 0.5)
@@
 	)
 	(segment
-		(start 122.775 54.45)
-		(end 125.15 53.425)
+		(start 111.12 56.75)
+		(end 113.645 59.275)
 		(width 0.5)
 		(layer "F.Cu")
@@
 	)
 	(segment
-		(start 130.125 95)
-		(end 130.15 94.975)
+		(start 127.7375 53.4875)
+		(end 129.275 55.025)
+		(width 0.5)
+		(layer "F.Cu")
+		(net 8)
+	)
+	(segment
+		(start 123.625 53.4875)
+		(end 127.7375 53.4875)
 		(width 0.5)
 		(layer "F.Cu")
@@
 	)
 	(segment
-		(start 112.625 59.125)
-		(end 119.8 59)
+		(start 132.225 94.55)
+		(end 134.14 94.55)
 		(width 0.5)
 		(layer "F.Cu")
@@
 	)
 	(segment
+		(start 130.025 94.9)
+		(end 131.875 94.9)
+		(width 0.5)
+		(layer "F.Cu")
+		(net 8)
+	)
+	(segment
 		(start 131.875 94.9)
-		(end 130.125 95)
+		(end 132.225 94.55)
 		(width 0.5)
 		(layer "F.Cu")
@@
 	)
 	(segment
-		(start 111.12 56.75)
-		(end 112.625 59.125)
+		(start 120.075 55.575)
+		(end 122.075 53.575)
 		(width 0.5)
 		(layer "F.Cu")
@@
 	)
 	(via
-		(at 130.15 94.975)
+		(at 129.925 94.8)
 		(size 0.5)
 		(drill 0.3)
@@
 	)
 	(segment
-		(start 128.875 92.875)
+		(start 128.934107 93.809107)
 		(end 128.934107 81.625)
 		(width 0.5)
@@
 	)
 	(segment
-		(start 130.15 94.975)
-		(end 128.875 92.875)
+		(start 129.925 94.8)
+		(end 128.934107 93.809107)
 		(width 0.5)
 		(layer "B.Cu")
@@
 	)
 	(segment
+		(start 118.775 87.607396)
+		(end 118.782396 87.6)
+		(width 0.5)
+		(layer "F.Cu")
+		(net 10)
+	)
+	(segment
+		(start 119.352616 76.05)
+		(end 119.4 76.097384)
+		(width 0.5)
+		(layer "F.Cu")
+		(net 10)
+	)
+	(segment
 		(start 119.4 76.097384)
 		(end 121.475 76.025)
@@
 	)
 	(segment
-		(start 117.175 76.175)
-		(end 119.4 76.097384)
+		(start 118.782396 87.6)
+		(end 120.9 87.6)
 		(width 0.5)
 		(layer "F.Cu")
@@
 	)
 	(segment
+		(start 117.3 76.05)
+		(end 119.352616 76.05)
+		(width 0.5)
+		(layer "F.Cu")
+		(net 10)
+	)
+	(segment
 		(start 119.4 76.097384)
 		(end 119.4 77.75)
@@
 	)
 	(segment
-		(start 118.775 87.607396)
-		(end 118.775 86.025)
+		(start 117.175 76.175)
+		(end 117.3 76.05)
 		(width 0.5)
 		(layer "F.Cu")
@@
 	)
 	(segment
-		(start 118.775 87.607396)
+		(start 120.9 87.6)
 		(end 121.1 87.8)
 		(width 0.5)
@@
 	)
 	(segment
+		(start 118.775 87.607396)
+		(end 118.775 86.025)
+		(width 0.5)
+		(layer "F.Cu")
+		(net 10)
+	)
+	(segment
 		(start 135.415 89.105)
 		(end 135.4 87.175)
@@
 	)
 	(segment
-		(start 125.175 55.35)
-		(end 125.15 55.325)
+		(start 123.65 55.4125)
+		(end 123.625 55.3875)
 		(width 0.5)
 		(layer "F.Cu")
@@
 	)
 	(segment
-		(start 125.175 58.025)
-		(end 125.175 55.35)
+		(start 123.65 58.0875)
+		(end 123.65 55.4125)
 		(width 0.5)
 		(layer "F.Cu")
